File: LED_Display/POV_PCB.kicad_sch (KiCad schematic)
At the start: 10 parts, among them U11 A3144

Commit message: AddComponant
Parts:
- C16, C7: footprint (none) -> Capacitor_THT:CP_Radial_D10.0mm_P5.00mm
Changed lines of the file:
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@@
 			)
 		)
-		(property "Footprint" ""
+		(property "Footprint" "Capacitor_THT:CP_Radial_D10.0mm_P5.00mm"
 			(at 225.7552 113.03 0)
 			(hide yes)
@@
 			)
 		)
-		(property "Footprint" ""
+		(property "Footprint" "Capacitor_THT:CP_Radial_D10.0mm_P5.00mm"
 			(at 238.4552 113.03 0)
 			(hide yes)
