File: LED_DisplayV1/LED_DisplayV1.kicad_pcb (KiCad board)
At the start: 2 copper layers, 100 x 100 mm, 105 parts, among them U10 TPIC6C595N, U3 TPIC6C595N, U4 TPIC6C595N, U5 TPIC6C595N, U6 TPIC6C595N, U7 TPIC6C595N, U8 TPIC6C595N, U9 TPIC6C595N

Commit message: Start_Routing_DisplayBoard
Parts:
- removed C14, C15, C17, C18, C19, C20, C21, C22: 0.1uF, Capacitor_SMD:C_0603_1608Metric_Pad1.08x0.95mm_HandSolder
- removed C16: 220uF, Capacitor_THT:CP_Radial_D10.0mm_P5.00mm
- removed the D18 at (235.2, 99.0)
- removed the D19 at (235.2, 102.7)
- removed the D20 at (235.2, 106.3)
- removed D69, D70: 1N5818, Diode_THT:D_DO-41_SOD81_P10.16mm_Horizontal
- removed LED2: LED_line, my_footprints:LED_line_2.0_l
- removed R11, R12, R13, R14, R15, R16, R17, R18: 10k, Resistor_SMD:R_0402_1005Metric_Pad0.72x0.64mm_HandSolder
- removed U10: TPIC6C595N, TPIC6C595N:N0016A
- added C1: 220uF, Capacitor_THT:CP_Radial_D10.0mm_P5.00mm, F.Cu at (170.0, 127.0)
- added C10: 0.1uF, Capacitor_SMD:C_0603_1608Metric_Pad1.08x0.95mm_HandSolder, F.Cu at (97.6, 112.5)
- added C2: 220uF, Capacitor_THT:CP_Radial_D10.0mm_P5.00mm, F.Cu at (135.0, 127.0)
- added C3: 0.1uF, Capacitor_SMD:C_0603_1608Metric_Pad1.08x0.95mm_HandSolder, F.Cu at (140.6, 66.0)
- added C4: 0.1uF, Capacitor_SMD:C_0603_1608Metric_Pad1.08x0.95mm_HandSolder, F.Cu at (122.1, 51.0)
- added C5: 0.1uF, Capacitor_SMD:C_0603_1608Metric_Pad1.08x0.95mm_HandSolder, F.Cu at (192.1, 75.0)
- added C6: 0.1uF, Capacitor_SMD:C_0603_1608Metric_Pad1.08x0.95mm_HandSolder, F.Cu at (157.6, 68.0)
- added C8: 0.1uF, Capacitor_SMD:C_0603_1608Metric_Pad1.08x0.95mm_HandSolder, F.Cu at (201.6, 87.0)
- added C9: 0.1uF, Capacitor_SMD:C_0603_1608Metric_Pad1.08x0.95mm_HandSolder, F.Cu at (105.1, 91.5)
- added D1: 1N5818, Diode_THT:D_DO-41_SOD81_P10.16mm_Horizontal, F.Cu at (172.5, 139.9)
- added D2: 1N5818, Diode_THT:D_DO-41_SOD81_P10.16mm_Horizontal, F.Cu at (167.0, 150.0)
- added D4: 1N5818, Diode_THT:D_DO-41_SOD81_P10.16mm_Horizontal, F.Cu at (129.0, 150.0)
- added D51: LED, LED_THT:LED_Rectangular_W3.0mm_H2.0mm, F.Cu at (167.5, 108.7)
- added D52: LED, LED_THT:LED_Rectangular_W3.0mm_H2.0mm, F.Cu at (165.2, 107.3)
- added L1: Coil, my_footprints:coil_large, F.Cu at (150.0, 100.0)
- added R1: 20k, Resistor_THT:R_Axial_DIN0207_L6.3mm_D2.5mm_P10.16mm_Horizontal, F.Cu at (162.0, 151.1)
- added R3: 10k, Resistor_SMD:R_0402_1005Metric_Pad0.72x0.64mm_HandSolder, F.Cu at (137.4, 71.0)
- added R4: 10k, Resistor_SMD:R_0402_1005Metric_Pad0.72x0.64mm_HandSolder, F.Cu at (138.1, 48.0)
- added R5: 10k, Resistor_SMD:R_0402_1005Metric_Pad0.72x0.64mm_HandSolder, F.Cu at (141.4, 73.0)
- added R6: 10k, Resistor_SMD:R_0402_1005Metric_Pad0.72x0.64mm_HandSolder, F.Cu at (201.9, 80.5)
- added R7: 10k, Resistor_SMD:R_0402_1005Metric_Pad0.72x0.64mm_HandSolder, F.Cu at (177.0, 95.4)
- added R8: 10k, Resistor_SMD:R_0402_1005Metric_Pad0.72x0.64mm_HandSolder, F.Cu at (104.1, 82.5)
- added R9: 10k, Resistor_SMD:R_0402_1005Metric_Pad0.72x0.64mm_HandSolder, F.Cu at (106.4, 100.0)
- added U2: TPIC6C595N, TPIC6C595N:N0016A, F.Cu at (149.2, 51.1)
- C7: value 220uF -> 0.1uF; footprint Capacitor_THT:CP_Radial_D10.0mm_P5.00mm -> Capacitor_SMD:C_0603_1608Metric_Pad1.08x0.95mm_HandSolder
- D68: value 1N5818 -> LED; footprint Diode_THT:D_DO-41_SOD81_P10.16mm_Horizontal -> LED_THT:LED_Rectangular_W3.0mm_H2.0mm
- R2: value 20k -> 10k; footprint Resistor_THT:R_Axial_DIN0207_L6.3mm_D2.5mm_P10.16mm_Horizontal -> Resistor_SMD:R_0402_1005Metric_Pad0.72x0.64mm_HandSolder
- moved U6 177.2 mm to (201.7, 99.8)
- moved RN4 162.3 mm to (172.5, 73.0), turned to -150 degrees
- moved D25 152.1 mm to (188.7, 76.2), turned to -60 degrees
- moved D26 150.2 mm to (186.3, 77.6), turned to -60 degrees
- moved D27 148.4 mm to (184.0, 78.9), turned to -60 degrees
- moved D28 146.6 mm to (181.7, 80.3), turned to -60 degrees
- moved D29 144.8 mm to (179.4, 81.6), turned to -60 degrees
- moved D30 143.1 mm to (177.0, 82.9), turned to -60 degrees
- moved U3 142.9 mm to (130.2, 54.1)
- moved D31 141.5 mm to (174.7, 84.3), turned to -60 degrees
- moved D20 136.4 mm to (101.2, 70.3), turned to -120 degrees
- moved D53 134.5 mm to (100.7, 127.0), turned to -60 degrees
- moved U5 133.6 mm to (149.2, 73.4)
- moved D19 131.8 mm to (103.5, 71.7), turned to -120 degrees
- moved D46 128.8 mm to (179.2, 115.4), turned to -120 degrees
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- renumbered D16 to D10, D17 to D11, D52 to D12, D4 to D13, D5 to D14, D6 to D15, D7 to D16, D8 to D17, D9 to D18, D10 to D19, D51 to D20, D11 to D5, D12 to D6, D13 to D7, D14 to D8, D15 to D9
Connections:
- C7 pad 1: /LED1/V_led -> /LED1/+5V
- D10 pad 1: Net-(D16-K) -> Net-(D10-K)
- D10 pad 2: Net-(D16-A) -> Net-(D10-A)
- D11 pad 1: Net-(D17-K) -> Net-(D11-K)
- D11 pad 2: Net-(D17-A) -> Net-(D11-A)
- D12 pad 1: Net-(D52-K) -> Net-(D12-K)
- D12 pad 2: Net-(D52-A) -> Net-(D12-A)
- D13 pad 1: Net-(D4-K) -> Net-(D13-K)
- D13 pad 2: Net-(D4-A) -> Net-(D13-A)
- D14 pad 1: Net-(D5-K) -> Net-(D14-K)
- D14 pad 2: Net-(D5-A) -> Net-(D14-A)
- D15 pad 1: Net-(D6-K) -> Net-(D15-K)
- D15 pad 2: Net-(D6-A) -> Net-(D15-A)
- D16 pad 1: Net-(D7-K) -> Net-(D16-K)
- D16 pad 2: Net-(D7-A) -> Net-(D16-A)
- D17 pad 1: Net-(D8-K) -> Net-(D17-K)
- D17 pad 2: Net-(D8-A) -> Net-(D17-A)
- D18 pad 1: Net-(D9-K) -> Net-(D18-K)
- D18 pad 2: Net-(D9-A) -> Net-(D18-A)
- D19 pad 1: Net-(D10-K) -> Net-(D19-K)
- D19 pad 2: Net-(D10-A) -> Net-(D19-A)
- D20 pad 1: Net-(D51-K) -> Net-(D20-K)
- D20 pad 2: Net-(D51-A) -> Net-(D20-A)
- D3 pad 1: Net-(D3-K) -> /LED1/V_led
- D3 pad 2: GND -> Net-(D3-A)
- D5 pad 1: Net-(D11-K) -> Net-(D5-K)
- D5 pad 2: Net-(D11-A) -> Net-(D5-A)
- D6 pad 1: Net-(D12-K) -> Net-(D6-K)
- D6 pad 2: Net-(D12-A) -> Net-(D6-A)
- D68 pad 1: /LED1/V_led -> Net-(D68-K)
- D68 pad 2: Net-(D3-K) -> Net-(D68-A)
- D7 pad 1: Net-(D13-K) -> Net-(D7-K)
- D7 pad 2: Net-(D13-A) -> Net-(D7-A)
- D8 pad 1: Net-(D14-K) -> Net-(D8-K)
- D8 pad 2: Net-(D14-A) -> Net-(D8-A)
- D9 pad 1: Net-(D15-K) -> Net-(D9-K)
- D9 pad 2: Net-(D15-A) -> Net-(D9-A)
- R2 pad 1: Net-(A1-D2) -> /LED1/+5V
- R2 pad 2: /LED1/+5V -> Net-(U2-CLR_N)
- RN1 pad 2: Net-(D51-A) -> Net-(D5-A)
- RN1 pad 3: Net-(D4-A) -> Net-(D6-A)
- RN1 pad 4: Net-(D5-A) -> Net-(D7-A)
- RN1 pad 5: Net-(D6-A) -> Net-(D8-A)
- RN1 pad 6: Net-(D7-A) -> Net-(D9-A)
- RN1 pad 7: Net-(D8-A) -> Net-(D10-A)
- RN1 pad 8: Net-(D9-A) -> Net-(D11-A)
- RN1 pad 9: Net-(D10-A) -> Net-(D12-A)
- RN2 pad 2: Net-(D52-A) -> Net-(D13-A)
- RN2 pad 3: Net-(D11-A) -> Net-(D14-A)
- RN2 pad 4: Net-(D12-A) -> Net-(D15-A)
- RN2 pad 5: Net-(D13-A) -> Net-(D16-A)
- RN2 pad 6: Net-(D14-A) -> Net-(D17-A)
- RN2 pad 7: Net-(D15-A) -> Net-(D18-A)
- RN2 pad 8: Net-(D16-A) -> Net-(D19-A)
- RN2 pad 9: Net-(D17-A) -> Net-(D20-A)
- RN3 pad 2: Net-(D53-A) -> Net-(D21-A)
- RN3 pad 3: Net-(D18-A) -> Net-(D22-A)
- RN3 pad 4: Net-(D19-A) -> Net-(D23-A)
- RN3 pad 5: Net-(D20-A) -> Net-(D24-A)
- RN3 pad 6: Net-(D21-A) -> Net-(D25-A)
- RN3 pad 7: Net-(D22-A) -> Net-(D26-A)
- RN3 pad 8: Net-(D23-A) -> Net-(D27-A)
- RN3 pad 9: Net-(D24-A) -> Net-(D28-A)
- RN4 pad 2: Net-(D54-A) -> Net-(D29-A)
- RN4 pad 3: Net-(D25-A) -> Net-(D30-A)
- RN4 pad 4: Net-(D26-A) -> Net-(D31-A)
- RN4 pad 5: Net-(D27-A) -> Net-(D32-A)
- RN4 pad 6: Net-(D28-A) -> Net-(D33-A)
- RN4 pad 7: Net-(D29-A) -> Net-(D34-A)
- RN4 pad 8: Net-(D30-A) -> Net-(D35-A)
- RN4 pad 9: Net-(D31-A) -> Net-(D36-A)
- RN5 pad 2: Net-(D55-A) -> Net-(D44-A)
- RN5 pad 3: Net-(D32-A) -> Net-(D43-A)
- RN5 pad 4: Net-(D33-A) -> Net-(D42-A)
- RN5 pad 5: Net-(D34-A) -> Net-(D41-A)
- RN5 pad 6: Net-(D35-A) -> Net-(D40-A)
- RN5 pad 7: Net-(D36-A) -> Net-(D39-A)
- RN5 pad 8: Net-(D37-A) -> Net-(D38-A)
- RN5 pad 9: Net-(D38-A) -> Net-(D37-A)
- RN6 pad 2: Net-(D56-A) -> Net-(D52-A)
- RN6 pad 3: Net-(D39-A) -> Net-(D51-A)
- RN6 pad 4: Net-(D40-A) -> Net-(D50-A)
- RN6 pad 5: Net-(D41-A) -> Net-(D49-A)
- RN6 pad 6: Net-(D42-A) -> Net-(D48-A)
- RN6 pad 7: Net-(D43-A) -> Net-(D47-A)
- RN6 pad 8: Net-(D44-A) -> Net-(D46-A)
- RN7 pad 2: Net-(D57-A) -> Net-(D53-A)
- RN7 pad 3: Net-(D46-A) -> Net-(D54-A)
- RN7 pad 4: Net-(D47-A) -> Net-(D55-A)
- RN7 pad 5: Net-(D48-A) -> Net-(D56-A)
- RN7 pad 6: Net-(D49-A) -> Net-(D57-A)
- RN7 pad 7: Net-(D50-A) -> Net-(D58-A)
- RN7 pad 8: Net-(D58-A) -> Net-(D59-A)
- RN7 pad 9: Net-(D59-A) -> Net-(D60-A)
- RN8 pad 2: Net-(D60-A) -> Net-(D61-A)
- RN8 pad 3: Net-(D61-A) -> Net-(D62-A)
- RN8 pad 4: Net-(D62-A) -> Net-(D63-A)
- RN8 pad 5: Net-(D63-A) -> Net-(D64-A)
- RN8 pad 6: Net-(D64-A) -> Net-(D65-A)
- RN8 pad 7: Net-(D65-A) -> Net-(D66-A)
- RN8 pad 8: Net-(D66-A) -> Net-(D67-A)
- RN8 pad 9: Net-(D67-A) -> Net-(D68-A)
- U3 pad 11: Net-(D7-K) -> Net-(D17-K)
- U3 pad 12: Net-(D8-K) -> Net-(D18-K)
- U3 pad 13: Net-(D9-K) -> Net-(D19-K)
- U3 pad 14: Net-(D10-K) -> Net-(D20-K)
- U3 pad 2: /LED1/SER_IN -> /LED1/Ser_out
- U3 pad 3: Net-(D51-K) -> Net-(D13-K)
- U3 pad 4: Net-(D4-K) -> Net-(D14-K)
- U3 pad 5: Net-(D5-K) -> Net-(D15-K)
- U3 pad 6: Net-(D6-K) -> Net-(D16-K)
- U3 pad 9: /LED1/Ser_out -> /LED2/Ser_out
- U4 pad 11: Net-(D14-K) -> Net-(D25-K)
- U4 pad 12: Net-(D15-K) -> Net-(D26-K)
- U4 pad 13: Net-(D16-K) -> Net-(D27-K)
- U4 pad 14: Net-(D17-K) -> Net-(D28-K)
- U4 pad 2: /LED1/Ser_out -> /LED2/Ser_out
- U4 pad 3: Net-(D52-K) -> Net-(D21-K)
- U4 pad 4: Net-(D11-K) -> Net-(D22-K)
- U4 pad 5: Net-(D12-K) -> Net-(D23-K)
- U4 pad 6: Net-(D13-K) -> Net-(D24-K)
- U4 pad 9: /LED2/Ser_out -> /LED3/Ser_out
- U5 pad 11: Net-(D21-K) -> Net-(D33-K)
- U5 pad 12: Net-(D22-K) -> Net-(D34-K)
- U5 pad 13: Net-(D23-K) -> Net-(D35-K)
- U5 pad 14: Net-(D24-K) -> Net-(D36-K)
- U5 pad 2: /LED2/Ser_out -> /LED3/Ser_out
- U5 pad 3: Net-(D53-K) -> Net-(D29-K)
- U5 pad 4: Net-(D18-K) -> Net-(D30-K)
- U5 pad 5: Net-(D19-K) -> Net-(D31-K)
- U5 pad 6: Net-(D20-K) -> Net-(D32-K)
- U5 pad 9: /LED3/Ser_out -> /LED4/Ser_out
- U6 pad 11: Net-(D28-K) -> Net-(D40-K)
- U6 pad 12: Net-(D29-K) -> Net-(D39-K)
- U6 pad 13: Net-(D30-K) -> Net-(D38-K)
- U6 pad 14: Net-(D31-K) -> Net-(D37-K)
- U6 pad 2: /LED3/Ser_out -> /LED4/Ser_out
- U6 pad 3: Net-(D54-K) -> Net-(D44-K)
- U6 pad 4: Net-(D25-K) -> Net-(D43-K)
- U6 pad 5: Net-(D26-K) -> Net-(D42-K)
- U6 pad 6: Net-(D27-K) -> Net-(D41-K)
- U6 pad 9: /LED4/Ser_out -> /LED5/Ser_out
- U7 pad 11: Net-(D35-K) -> Net-(D48-K)
- U7 pad 12: Net-(D36-K) -> Net-(D47-K)
- U7 pad 13: Net-(D37-K) -> Net-(D46-K)
- U7 pad 14: Net-(D38-K) -> Net-(D45-K)
- U7 pad 2: /LED4/Ser_out -> /LED5/Ser_out
- U7 pad 3: Net-(D55-K) -> Net-(D52-K)
- U7 pad 4: Net-(D32-K) -> Net-(D51-K)
- U7 pad 5: Net-(D33-K) -> Net-(D50-K)
- U7 pad 6: Net-(D34-K) -> Net-(D49-K)
- U7 pad 9: /LED5/Ser_out -> /LED6/Ser_out
- U8 pad 11: Net-(D42-K) -> Net-(D57-K)
- U8 pad 12: Net-(D43-K) -> Net-(D58-K)
- U8 pad 13: Net-(D44-K) -> Net-(D59-K)
- U8 pad 14: Net-(D45-K) -> Net-(D60-K)
- U8 pad 2: /LED5/Ser_out -> /LED6/Ser_out
- U8 pad 3: Net-(D56-K) -> Net-(D53-K)
- U8 pad 4: Net-(D39-K) -> Net-(D54-K)
- U8 pad 5: Net-(D40-K) -> Net-(D55-K)
- U8 pad 6: Net-(D41-K) -> Net-(D56-K)
- U8 pad 9: /LED6/Ser_out -> /LED7/Ser_out
- U9 pad 11: Net-(D49-K) -> Net-(D65-K)
- U9 pad 12: Net-(D50-K) -> Net-(D66-K)
- U9 pad 13: Net-(D58-K) -> Net-(D67-K)
- U9 pad 14: Net-(D59-K) -> Net-(D68-K)
- U9 pad 2: /LED6/Ser_out -> /LED7/Ser_out
- U9 pad 3: Net-(D57-K) -> Net-(D61-K)
- U9 pad 4: Net-(D46-K) -> Net-(D62-K)
- U9 pad 5: Net-(D47-K) -> Net-(D63-K)
- U9 pad 6: Net-(D48-K) -> Net-(D64-K)
- U9 pad 9: /LED7/Ser_out -> /LED8/Ser_out
Routing:
- net GND: track 0.00 -> 191.8 mm
- net /LED1/V_led: track 0.00 -> 139.2 mm
- net /LED1/+5V: track 0.00 -> 100.1 mm
- net Net-(D3-A): track 0.00 -> 36.0 mm
- net Net-(D1-A): track 0.00 -> 35.5 mm
- net Net-(D45-K): track 0.00 -> 29.3 mm
- net Net-(D46-K): track 0.00 -> 26.7 mm
- net Net-(D47-K): track 0.00 -> 24.4 mm
- net Net-(D52-K): track 0.00 -> 19.9 mm
- net Net-(D48-K): track 0.00 -> 17.3 mm
- net Net-(D51-K): track 0.00 -> 17.1 mm
- net Net-(D50-K): track 0.00 -> 14.2 mm
- net Net-(D61-K): track 0.00 -> 13.7 mm
- net Net-(D62-K): track 0.00 -> 12.3 mm
- net Net-(D49-K): track 0.00 -> 11.7 mm
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Other:
- board size 100 x 100 mm -> 120 x 120 mm

Commit message: All_wired
Parts:
- removed A1: Arduino_Nano_ESP32, Module:Arduino_Nano
- removed the C10 at (97.6, 112.5)
- removed the C9 at (105.1, 91.5)
- removed the D10 at (124.5, 83.8)
- removed the D11 at (122.2, 82.4)
- removed the D12 at (119.8, 81.1)
- removed the D13 at (117.5, 79.7)
- removed the D14 at (115.2, 78.4)
- removed the D15 at (112.8, 77.1)
- removed the D16 at (110.5, 75.7)
- removed the D17 at (108.2, 74.4)
- removed the D18 at (105.9, 73.0)
- removed the D19 at (103.5, 71.7)
- removed the D20 at (101.2, 70.3)
- removed the D5 at (136.1, 90.5)
- removed the D6 at (133.8, 89.1)
- removed the D7 at (131.5, 87.8)
- removed the D8 at (129.1, 86.5)
- removed the D9 at (126.8, 85.1)
- removed R2, R3, R4, R5, R6, R7, R8, R9: 10k, Resistor_SMD:R_0402_1005Metric_Pad0.72x0.64mm_HandSolder
- removed the RN7 at (97.4, 121.7)
- removed the RN8 at (118.0, 125.0)
- removed the U8 at (98.2, 98.1)
- removed the U9 at (122.1, 99.3)
- added ?: , , F.Cu at (188.0, 72.0)
- added A2: Arduino_Nano_v3.x, Module:Arduino_Nano, F.Cu at (142.5, 117.0)
- added C11: 22uF, Capacitor_Tantalum_SMD:CP_EIA-3528-12_Kemet-T_HandSolder, F.Cu at (150.0, 74.5)
- added C12: 100nF, Capacitor_SMD:C_0603_1608Metric_Pad1.08x0.95mm_HandSolder, F.Cu at (150.0, 72.0)
- added C13: 1uF, Capacitor_SMD:C_0805_2012Metric_Pad1.18x1.45mm_HandSolder, F.Cu at (132.0, 136.0)
- added C7: 0.1uF, Capacitor_SMD:C_0603_1608Metric_Pad1.08x0.95mm_HandSolder, F.Cu at (156.5, 59.5)
- added C8: 0.1uF, Capacitor_SMD:C_0603_1608Metric_Pad1.08x0.95mm_HandSolder, F.Cu at (166.5, 49.5)
- added D53: LED, LED_THT:LED_Rectangular_W3.0mm_H2.0mm, F.Cu at (183.8, 118.0)
- added D54: LED, LED_THT:LED_Rectangular_W3.0mm_H2.0mm, F.Cu at (186.1, 119.4)
- added D55: LED, LED_THT:LED_Rectangular_W3.0mm_H2.0mm, F.Cu at (188.5, 120.7)
- added D56: LED, LED_THT:LED_Rectangular_W3.0mm_H2.0mm, F.Cu at (190.8, 122.1)
- added D57: LED, LED_THT:LED_Rectangular_W3.0mm_H2.0mm, F.Cu at (193.1, 123.4)
- added D58: LED, LED_THT:LED_Rectangular_W3.0mm_H2.0mm, F.Cu at (195.5, 124.8)
- added D59: LED, LED_THT:LED_Rectangular_W3.0mm_H2.0mm, F.Cu at (197.8, 126.1)
- added D60: LED, LED_THT:LED_Rectangular_W3.0mm_H2.0mm, F.Cu at (200.1, 127.5)
- added D61: LED, LED_THT:LED_Rectangular_W3.0mm_H2.0mm, F.Cu at (165.2, 107.3)
- added D62: LED, LED_THT:LED_Rectangular_W3.0mm_H2.0mm, F.Cu at (167.5, 108.6)
- added D63: LED, LED_THT:LED_Rectangular_W3.0mm_H2.0mm, F.Cu at (169.9, 110.0)
- added D64: LED, LED_THT:LED_Rectangular_W3.0mm_H2.0mm, F.Cu at (172.2, 111.3)
- added D65: LED, LED_THT:LED_Rectangular_W3.0mm_H2.0mm, F.Cu at (174.5, 112.7)
- added D66: LED, LED_THT:LED_Rectangular_W3.0mm_H2.0mm, F.Cu at (176.8, 114.0)
- added D67: LED, LED_THT:LED_Rectangular_W3.0mm_H2.0mm, F.Cu at (179.2, 115.4)
- added D68: LED, LED_THT:LED_Rectangular_W3.0mm_H2.0mm, F.Cu at (181.5, 116.7)
- added RN5: R_Network08, Resistor_THT:R_Array_SIP9, F.Cu at (161.0, 86.5)
- added RN6: R_Network08, Resistor_THT:R_Array_SIP9, F.Cu at (176.0, 72.0)
- added U1: A3144, my_footprints:A3144, F.Cu at (150.0, 154.0)
- added U10: AMS1117-5.0, Package_TO_SOT_SMD:SOT-223-3_TabPin2, F.Cu at (150.0, 80.0)
- added U6: TPIC6C595N, TPIC6C595N:N0016A, F.Cu at (162.0, 69.0)
- added U7: TPIC6C595N, TPIC6C595N:N0016A, F.Cu at (172.0, 59.0)
- moved D28 81.2 mm to (101.1, 70.3), turned to -120 degrees
- moved D21 81.1 mm to (117.4, 79.7), turned to -120 degrees
- moved D27 80.9 mm to (103.4, 71.6), turned to -120 degrees
- moved D22 80.8 mm to (115.1, 78.4), turned to -120 degrees
- moved D26 80.7 mm to (105.8, 73.0), turned to -120 degrees
- moved D23 80.6 mm to (112.8, 77.0), turned to -120 degrees
- moved D25 80.6 mm to (108.1, 74.3), turned to -120 degrees
- moved D24 80.6 mm to (110.4, 75.7), turned to -120 degrees
- moved RN3 68.7 mm to (124.5, 72.0), turned to 150 degrees
- moved C5 64.0 mm to (133.5, 49.5), turned to -30 degrees
- moved U3 59.1 mm to (116.0, 100.0)
- moved RN1 56.9 mm to (98.5, 123.5), turned to 30 degrees
- moved U2 54.9 mm to (100.0, 100.0)
- moved RN2 54.9 mm to (118.5, 125.0), turned to 30 degrees
- moved D37 50.4 mm to (179.4, 81.6), turned to -60 degrees
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- renumbered C7 to C10, C8 to C9, D58 to D10, D59 to D11, D60 to D12, D61 to D13, D62 to D14, D63 to D15, D64 to D16, D65 to D17, D66 to D18, D67 to D19, D68 to D20, D53 to D5, D54 to D6, D55 to D7, D56 to D8, D57 to D9, RN5 to RN7, RN6 to RN8, U3 to U2, U2 to U3, U6 to U8, U7 to U9
Connections:
- C1 pad 1: /LED1/V_led -> Net-(A2-VIN)
- C2 pad 1: /LED1/V_led -> Net-(A2-VIN)
- D1 pad 1: /LED1/V_led -> Net-(A2-VIN)
- D10 pad 1: Net-(D58-K) -> Net-(D10-K)
- D10 pad 2: Net-(D58-A) -> Net-(D10-A)
- D11 pad 1: Net-(D59-K) -> Net-(D11-K)
- D11 pad 2: Net-(D59-A) -> Net-(D11-A)
- D12 pad 1: Net-(D60-K) -> Net-(D12-K)
- D12 pad 2: Net-(D60-A) -> Net-(D12-A)
- D13 pad 1: Net-(D61-K) -> Net-(D13-K)
- D13 pad 2: Net-(D61-A) -> Net-(D13-A)
- D14 pad 1: Net-(D62-K) -> Net-(D14-K)
- D14 pad 2: Net-(D62-A) -> Net-(D14-A)
- D15 pad 1: Net-(D63-K) -> Net-(D15-K)
- D15 pad 2: Net-(D63-A) -> Net-(D15-A)
- D16 pad 1: Net-(D64-K) -> Net-(D16-K)
- D16 pad 2: Net-(D64-A) -> Net-(D16-A)
- D17 pad 1: Net-(D65-K) -> Net-(D17-K)
- D17 pad 2: Net-(D65-A) -> Net-(D17-A)
- D18 pad 1: Net-(D66-K) -> Net-(D18-K)
- D18 pad 2: Net-(D66-A) -> Net-(D18-A)
- D19 pad 1: Net-(D67-K) -> Net-(D19-K)
- D19 pad 2: Net-(D67-A) -> Net-(D19-A)
- D20 pad 1: Net-(D68-K) -> Net-(D20-K)
- D20 pad 2: Net-(D68-A) -> Net-(D20-A)
- D3 pad 1: /LED1/V_led -> Net-(A2-VIN)
- D5 pad 1: Net-(D53-K) -> Net-(D5-K)
- D5 pad 2: Net-(D53-A) -> Net-(D5-A)
- D6 pad 1: Net-(D54-K) -> Net-(D6-K)
- D6 pad 2: Net-(D54-A) -> Net-(D6-A)
- D7 pad 1: Net-(D55-K) -> Net-(D7-K)
- D7 pad 2: Net-(D55-A) -> Net-(D7-A)
- D8 pad 1: Net-(D56-K) -> Net-(D8-K)
- D8 pad 2: Net-(D56-A) -> Net-(D8-A)
- D9 pad 1: Net-(D57-K) -> Net-(D9-K)
- D9 pad 2: Net-(D57-A) -> Net-(D9-A)
- R1 pad 2: /LED1/+5V -> Net-(A2-+5V)
- RN1 pad 1: /LED1/V_led -> /LED1/+5V
- RN2 pad 1: /LED1/V_led -> /LED1/+5V
- RN3 pad 1: /LED1/V_led -> /LED1/+5V
- RN4 pad 1: /LED1/V_led -> /LED1/+5V
- RN7 pad 1: /LED1/V_led -> /LED1/+5V
- RN7 pad 2: Net-(D44-A) -> Net-(D53-A)
- RN7 pad 3: Net-(D43-A) -> Net-(D54-A)
- RN7 pad 4: Net-(D42-A) -> Net-(D55-A)
- RN7 pad 5: Net-(D41-A) -> Net-(D56-A)
- RN7 pad 6: Net-(D40-A) -> Net-(D57-A)
- RN7 pad 7: Net-(D39-A) -> Net-(D58-A)
- RN7 pad 8: Net-(D38-A) -> Net-(D59-A)
- RN7 pad 9: Net-(D37-A) -> Net-(D60-A)
- RN8 pad 1: /LED1/V_led -> /LED1/+5V
- RN8 pad 2: Net-(D52-A) -> Net-(D61-A)
- RN8 pad 3: Net-(D51-A) -> Net-(D62-A)
- RN8 pad 4: Net-(D50-A) -> Net-(D63-A)
- RN8 pad 5: Net-(D49-A) -> Net-(D64-A)
- RN8 pad 6: Net-(D48-A) -> Net-(D65-A)
- RN8 pad 7: Net-(D47-A) -> Net-(D66-A)
- RN8 pad 8: Net-(D46-A) -> Net-(D67-A)
- RN8 pad 9: Net-(D45-A) -> Net-(D68-A)
- U2 pad 11: Net-(D17-K) -> Net-(D9-K)
- U2 pad 12: Net-(D18-K) -> Net-(D10-K)
- U2 pad 13: Net-(D19-K) -> Net-(D11-K)
- U2 pad 14: Net-(D20-K) -> Net-(D12-K)
- U2 pad 2: /LED1/Ser_out -> /LED1/SER_IN
- U2 pad 3: Net-(D13-K) -> Net-(D5-K)
- U2 pad 4: Net-(D14-K) -> Net-(D6-K)
- U2 pad 5: Net-(D15-K) -> Net-(D7-K)
- U2 pad 6: Net-(D16-K) -> Net-(D8-K)
- U2 pad 7: Net-(U3-CLR_N) -> /LED1/+5V
- U2 pad 9: /LED2/Ser_out -> /LED1/Ser_out
- U3 pad 11: Net-(D9-K) -> Net-(D17-K)
- U3 pad 12: Net-(D10-K) -> Net-(D18-K)
- U3 pad 13: Net-(D11-K) -> Net-(D19-K)
- U3 pad 14: Net-(D12-K) -> Net-(D20-K)
- U3 pad 2: /LED1/SER_IN -> /LED1/Ser_out
- U3 pad 3: Net-(D5-K) -> Net-(D13-K)
- U3 pad 4: Net-(D6-K) -> Net-(D14-K)
- U3 pad 5: Net-(D7-K) -> Net-(D15-K)
- U3 pad 6: Net-(D8-K) -> Net-(D16-K)
- U3 pad 7: Net-(U2-CLR_N) -> /LED1/+5V
- U3 pad 9: /LED1/Ser_out -> /LED2/Ser_out
- U4 pad 7: Net-(U4-CLR_N) -> /LED1/+5V
- U5 pad 7: Net-(U5-CLR_N) -> /LED1/+5V
- U8 pad 11: Net-(D40-K) -> Net-(D57-K)
- U8 pad 12: Net-(D39-K) -> Net-(D58-K)
- U8 pad 13: Net-(D38-K) -> Net-(D59-K)
- U8 pad 14: Net-(D37-K) -> Net-(D60-K)
- U8 pad 2: /LED4/Ser_out -> /LED6/Ser_out
- U8 pad 3: Net-(D44-K) -> Net-(D53-K)
- U8 pad 4: Net-(D43-K) -> Net-(D54-K)
- U8 pad 5: Net-(D42-K) -> Net-(D55-K)
- U8 pad 6: Net-(D41-K) -> Net-(D56-K)
- U8 pad 7: Net-(U6-CLR_N) -> /LED1/+5V
- U8 pad 9: /LED5/Ser_out -> /LED7/Ser_out
- U9 pad 11: Net-(D48-K) -> Net-(D65-K)
- U9 pad 12: Net-(D47-K) -> Net-(D66-K)
- U9 pad 13: Net-(D46-K) -> Net-(D67-K)
- U9 pad 14: Net-(D45-K) -> Net-(D68-K)
- U9 pad 2: /LED5/Ser_out -> /LED7/Ser_out
- U9 pad 3: Net-(D52-K) -> Net-(D61-K)
- U9 pad 4: Net-(D51-K) -> Net-(D62-K)
- U9 pad 5: Net-(D50-K) -> Net-(D63-K)
- U9 pad 6: Net-(D49-K) -> Net-(D64-K)
- U9 pad 7: Net-(U7-CLR_N) -> /LED1/+5V
- U9 pad 9: /LED6/Ser_out -> /LED8/Ser_out
Routing:
- net /LED1/+5V: track 100.1 -> 543.3 mm
- net /LED1/G: track 0.00 -> 342.7 mm, vias 0 -> 12
- net /LED1/RCK: track 0.00 -> 333.5 mm, vias 0 -> 10
- net /LED1/SRCK: track 0.00 -> 325.3 mm, vias 0 -> 5
- net GND: track 191.8 -> 389.0 mm, vias 0 -> 1
- net /LED1/V_led: track 139.2 -> 0.00 mm
- net Net-(A2-VIN): track 0.00 -> 120.8 mm
- net /LED1/SER_IN: track 0.00 -> 94.1 mm
- net /LED2/Ser_out: track 0.00 -> 91.6 mm, vias 0 -> 3
- net /LED4/Ser_out: track 0.00 -> 56.2 mm, vias 0 -> 2
- net Net-(A2-+5V): track 0.00 -> 51.1 mm
- net Net-(A2-D2): track 0.00 -> 46.8 mm
- net Net-(D28-K): track 0.00 -> 44.5 mm
- net /LED7/Ser_out: track 0.00 -> 44.0 mm
- net Net-(D27-K): track 0.00 -> 39.9 mm
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- added copper zone on B.Cu, net GND
- added copper zone on F.Cu, net GND

Commit message: ChangeCPosition
Parts:
- moved C13 10.2 mm to (134.0, 126.0)
- moved C1 6.00 mm to (170.0, 133.0)
- moved C2 6.00 mm to (135.0, 133.0)
Routing:
- net GND: track 389.0 -> 393.1 mm, vias 1 -> 18
- net Net-(A2-VIN): track 120.8 -> 118.0 mm
- net Net-(D6-K): track 33.1 -> 32.2 mm
- net Net-(D5-K): track 35.9 -> 35.1 mm
