File: LED_DisplayV2/LED_DisplayV2.kicad_pcb (KiCad board)
At the start: 4 copper layers, 120 x 120 mm, 105 parts, among them U1 A3144, U10 AMS1117-5.0, U2 TPIC6C595N, U3 TPIC6C595N, U4 TPIC6C595N, U5 TPIC6C595N, U6 TPIC6C595N, U7 TPIC6C595N, U8 TPIC6C595N, U9 TPIC6C595N

Commit message: Temp
Parts:
- moved ? 2.12 mm to (182.0, 143.5)
Routing:
- net Net-(D1-A): track 17.2 -> 18.0 mm
Changed lines of the file:
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@@
 			(outputformat 1)
 			(mirror no)
-			(drillshape 1)
+			(drillshape 0)
 			(scaleselection 1)
-			(outputdirectory "")
+			(outputdirectory "../../JLCgerber/DIsplay2/")
 		)
 	)
@@
 	(footprint ""
 		(layer "F.Cu")
-		(at 180.5 142)
+		(at 182 143.5)
 		(property "Reference" ""
 			(at 0 0 0)
@@
 	)
 	(segment
-		(start 180.5 142)
-		(end 180.5 142.08)
+		(start 175.42 150.08)
+		(end 172.5 150.08)
 		(width 2)
 		(layer "In2.Cu")
@@
 	)
 	(segment
-		(start 180.5 142.08)
-		(end 172.5 150.08)
+		(start 182 143.5)
+		(end 175.42 150.08)
 		(width 2)
 		(layer "In2.Cu")
@@
 		)
 	)
+	(group ""
+		(members "1b5062a5-b216-49e4-8266-ba4fc5b68e2a" "248e0702-b52a-4b49-bc67-1ec42230dc5e"
+			"34c3fdc9-8980-4f12-b5d8-74dd917dfe5a" "562f6f92-ceb4-4d95-a46d-c22683edd5ad"
+			"88320b0f-f99c-491f-b00a-0ae1d01ef5c0" "98fd4ae4-712a-4508-a8c4-c42b5674b2bd"
+			"9e5ee379-365f-4061-b7f5-e9a84bf1e0c9" "d2c7e73f-1632-4e57-a09e-0d50b6292f23"
+			"dc5733cf-c7da-4e3c-a1d1-66342241b773"
+		)
+	)
