File: LED_DisplayV2/LED_DisplayV2.kicad_pcb (KiCad board)
At the start: 4 copper layers, 120 x 120 mm, 105 parts, among them U1 A3144, U10 AMS1117-5.0, U2 TPIC6C595N, U3 TPIC6C595N, U4 TPIC6C595N, U5 TPIC6C595N, U6 TPIC6C595N, U7 TPIC6C595N, U8 TPIC6C595N, U9 TPIC6C595N

Commit message: ReworkPM2
Parts:
- moved C13 1.00 mm to (132.5, 126.5)
Routing:
- net Net-(A2-+5V): track 50.1 -> 49.1 mm

Commit message: FinalV1
Parts:
- removed the ? at (112.0, 128.0)
- removed the ? at (188.0, 128.0)
- added ?: , , F.Cu at (108.5, 78.0)
- added ?: , , F.Cu at (191.5, 78.0)
- moved ? 6.50 mm to (120.5, 137.5)
- moved ? 4.61 mm to (179.5, 137.5)
Routing:
- net Net-(D1-A): track 17.2 -> 21.2 mm
- net Net-(D3-A): track 19.8 -> 23.0 mm
- net Net-(D9-A): track 16.3 -> 14.4 mm
- net Net-(A2-+5V): track 49.1 -> 50.3 mm
- net Net-(D56-A): track 14.5 -> 13.8 mm
- net Net-(D8-K): track 40.7 -> 40.0 mm
- net Net-(D12-A): track 15.3 -> 14.7 mm
- net GND: vias 10 -> 45
- added copper zone on B.Cu, net GND
- added copper zone on F.Cu, net GND
Other:
- outline, holes or cut-outs redrawn
- board text added: "L1"
