File: Royer_coil/Royer_coil.kicad_pcb (KiCad board)
At the start: 2 copper layers, 98 x 98 mm, 2 parts

Commit message: FinalV1
Parts:
- added ?: , , F.Cu at (179.5, 137.5)
- added ?: , , F.Cu at (108.5, 78.0)
- added ?: , , F.Cu at (120.5, 137.5)
- added ?: , , F.Cu at (191.5, 78.0)
Routing:
- net Net-(L**1-Pad1): track 2089.9 -> 2116.2 mm

Commit message: FinalV2
Parts:
- removed  : , my_footprints:Pin_2mm (x2)
Routing:
- net Net-(L**1-Pad1): track 2116.2 -> 2114.1 mm
Changed lines of the file:
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@@
 		(embedded_fonts no)
 	)
-	(footprint "my_footprints:Pin_2mm"
-		(layer "F.Cu")
-		(at 150.19 47.86)
-		(property "Reference" " "
-			(at 0 -1.651 0)
-			(layer "F.SilkS")
-			(effects
-				(font
-					(size 1 1)
-					(thickness 0.15)
-				)
-			)
-		)
-		(property "Value" " "
-			(at 0 -2.921 0)
-			(layer "F.Fab")
-			(effects
-				(font
-					(size 1 1)
-					(thickness 0.15)
-				)
-			)
-		)
-		(property "Datasheet" ""
-			(at 0 0 0)
-			(layer "F.Fab")
-			(hide yes)
-			(effects
-				(font
-					(size 1.27 1.27)
-				)
-			)
-		)
-		(property "Description" ""
-			(at 0 0 0)
-			(layer "F.Fab")
-			(hide yes)
-			(effects
-				(font
-					(size 1.27 1.27)
-				)
-			)
-		)
-		(attr through_hole)
-		(duplicate_pad_numbers_are_jumpers no)
-		(pad "1" thru_hole circle
-			(at -38.19 24.64)
-			(size 2.5 2.5)
-			(drill 1)
-			(layers "*.Cu" "*.Mask")
-			(remove_unused_layers no)
-			(net "Net-(L**1-Pad1)")
-		)
-		(embedded_fonts no)
-	)
-	(footprint "my_footprints:Pin_2mm"
-		(layer "F.Cu")
-		(at 153.19 47.86)
-		(property "Reference" " "
-			(at 0 -1.651 0)
-			(layer "F.SilkS")
-			(effects
-				(font
-					(size 1 1)
-					(thickness 0.15)
-				)
-			)
-		)
-		(property "Value" " "
-			(at 0 -2.921 0)
-			(layer "F.Fab")
-			(effects
-				(font
-					(size 1 1)
-					(thickness 0.15)
-				)
-			)
-		)
-		(property "Datasheet" ""
-			(at 0 0 0)
-			(layer "F.Fab")
-			(hide yes)
-			(effects
-				(font
-					(size 1.27 1.27)
-				)
-			)
-		)
-		(property "Description" ""
-			(at 0 0 0)
-			(layer "F.Fab")
-			(hide yes)
-			(effects
-				(font
-					(size 1.27 1.27)
-				)
-			)
-		)
-		(attr through_hole)
-		(duplicate_pad_numbers_are_jumpers no)
-		(pad "1" thru_hole circle
-			(at 34.81 24.64)
-			(size 2.5 2.5)
-			(drill 1)
-			(layers "*.Cu" "*.Mask")
-			(remove_unused_layers no)
-		)
-		(embedded_fonts no)
-	)
 	(footprint ""
 		(layer "F.Cu")
@@
 		(width 1.5)
 		(layer "F.Cu")
-		(net "Net-(L**1-Pad1)")
-	)
-	(segment
-		(start 113.149277 74.176383)
-		(end 112 72.5)
-		(width 1.5)
-		(layer "F.Cu")

Commit message: Fix1
Other:
- board text removed: "SEK1"
- board text removed: "SEK2"
Changed lines of the file:
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@@
 			(outputformat 1)
 			(mirror no)
-			(drillshape 1)
+			(drillshape 0)
 			(scaleselection 1)
-			(outputdirectory "")
+			(outputdirectory "../../PCB_Garber/Royer_coil/")
 		)
 	)
@@
 		(layer "Edge.Cuts")
 	)
-	(gr_text "SEK1"
-		(at 117.02 128.58 0)
-		(layer "F.SilkS")
-		(effects
-			(font
-				(size 1.5 1.5)
-				(thickness 0.15)
-			)
-		)
-	)
-	(gr_text "SEK2"
-		(at 183.01 128.49 0)
-		(layer "F.SilkS")
-		(effects
-			(font
-				(size 1.5 1.5)
-				(thickness 0.15)
-			)
-		)
-	)
 	(segment
