File: Power_and_MotorV2/Power_and_MotorV2.kicad_pcb (KiCad board)
At the start: 2 copper layers, 110 x 110 mm, 25 parts, among them J1 Barrel_Jack_Switch_Pin3Ring, M1 Motor_DC, Q1 BC337, Q2 BC337, SW1 SW_DPDT_x2, U1 LM317_TO-220, U2 Pin-Connector, U3 Pin-Connector, U4 Pin-Connector, U5 Pin-Connector, U6 Pin-Connector, U7 Pin-Connector

Commit message: Fix1
Routing:
- net Net-(C4-Pad1): track 22.8 -> 22.0 mm
Changed lines of the file:
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@@
 			(outputformat 1)
 			(mirror no)
-			(drillshape 1)
+			(drillshape 0)
 			(scaleselection 1)
-			(outputdirectory "")
+			(outputdirectory "../../PCB_Garber/PowerBoard/")
 		)
 	)
@@
 		(sheetname "/")
 		(sheetfile "Power_and_MotorV2.kicad_sch")
-		(units
-			(unit
-				(name "A")
-				(pins "1" "2")
-			)
-		)
 		(attr through_hole)
 		(duplicate_pad_numbers_are_jumpers no)
-		(fp_circle
-			(center 0 5.08)
-			(end 2.54 7.62)
-			(stroke
-				(width 0.12)
-				(type solid)
-			)
-			(fill no)
-			(layer "F.SilkS")
-		)
 		(fp_line
 			(start 1.27 1.27)
@@
 		(at 201 55.5 90)
 		(property "Reference" "RV1"
-			(at -10.541 3.033 90)
+			(at -4.5 -7.5 90)
 			(layer "F.SilkS")
 			(effects
@@
 	)
 	(segment
-		(start 203.361434 53.401419)
-		(end 203.361434 52.321419)
+		(start 202.5 54.262853)
+		(end 202.5 51.459985)
+		(width 1)
+		(layer "F.Cu")
+		(net "Net-(C4-Pad1)")
+	)
+	(segment
+		(start 202.5 51.459985)
+		(end 201.361434 50.321419)
 		(width 1)
 		(layer "F.Cu")
@@
 	)
 	(segment
-		(start 203.361434 52.321419)
-		(end 201.361434 50.321419)
-		(width 1)
-		(layer "F.Cu")
-		(net "Net-(C4-Pad1)")
-	)
-	(segment
 		(start 201.361434 55.401419)
-		(end 203.361434 53.401419)
+		(end 202.5 54.262853)
 		(width 1)
 		(layer "F.Cu")

Commit message: Final
Parts:
- SW1: footprint Button_Switch_THT:SW_CK_JS202011AQN_DPDT_Angled -> SW_footprint:SW_1101M2S3CQE2
- moved SW1 1.12 mm to (201.0, 72.5), turned to 0 degrees
Routing:
- net Net-(D1-K): track 77.1 -> 66.7 mm
- net Net-(D2-A): track 110.1 -> 111.9 mm
