File: Power_and_MotorV2/Power_and_MotorV2.kicad_sch (KiCad schematic)
At the start: 24 parts, among them M1 Motor_DC, Q1 BC337, Q2 BC337, SW1 SW_DPDT_x2, U1 LM317_TO-220, U2 Pin-Connector, U3 Pin-Connector, U4 Pin-Connector, U5 Pin-Connector, U6 Pin-Connector, U7 Pin-Connector

Commit message: FinalV1
Parts:
- C3, C4, C5: footprint (none) -> Capacitor_SMD:C_0603_1608Metric_Pad1.08x0.95mm_HandSolder
Changed lines of the file:
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@@
 			)
 		)
-		(property "Footprint" ""
+		(property "Footprint" "Capacitor_SMD:C_0603_1608Metric_Pad1.08x0.95mm_HandSolder"
 			(at 111.4552 120.65 0)
 			(hide yes)
@@
 			)
 		)
-		(property "Footprint" ""
+		(property "Footprint" "Capacitor_SMD:C_0603_1608Metric_Pad1.08x0.95mm_HandSolder"
 			(at 200.3552 107.95 0)
 			(hide yes)
@@
 			)
 		)
-		(property "Footprint" ""
+		(property "Footprint" "Capacitor_SMD:C_0603_1608Metric_Pad1.08x0.95mm_HandSolder"
 			(at 138.1252 140.97 0)
 			(hide yes)

Commit message: Final
Parts:
- SW1: footprint Button_Switch_THT:SW_CK_JS202011AQN_DPDT_Angled -> SW_footprint:SW_1101M2S3CQE2
Changed lines of the file:
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@@
 			)
 		)
-		(property "Footprint" "Button_Switch_THT:SW_CK_JS202011AQN_DPDT_Angled"
+		(property "Footprint" "SW_footprint:SW_1101M2S3CQE2"
 			(at 189.23 93.98 0)
 			(hide yes)
